Commit message: 2nd lab

File: urdf/my_robot.urdf (robot description, URDF)
Before this commit: robot erl1, 4 links, 3 joints
Joints:
- removed joint left_wheel joint
- removed joint right_wheel joint
- added joint left_wheel_joint: type continous, parent link_chassis, child left_wheel, origin xyz=-0.1 0.15 0 rpy=0 0 0, axis 0 1 0, limit effort=100 velocity=10
- added joint right_wheel_joint: type continous, parent link_chassis, child right_wheel, origin xyz=-0.1 -0.15 0 rpy=0 0 0, axis 0 1 0, limit effort=100 velocity=10
